Commit message: [slam and nav2] add rtabmap slam and nav2

File: MentorPi/src/simulations/mentorpi_description/urdf/ack.xacro (robot description, xacro)
@@ -177,5 +177,5 @@
     <axis xyz="0 0 0"/>
   </joint>
-  <link name="lidar_frame">
+  <!-- <link name="lidar_frame">
     <inertial>
       <origin rpy="0 0 0" xyz="8.65086433231368E-05 9.02624784523964E-05 -0.0183546134614858"/>
@@ -204,5 +204,5 @@
     <child link="lidar_frame"/>
     <axis xyz="0 0 0"/>
-  </joint>
+  </joint> -->
   <xacro:include filename="$(find mentorpi_description)/urdf/imu.urdf.xacro"/>
 </robot>
